File: hardware/HSLinkIsolate.kicad_pcb (KiCad board)
At the start: 2 copper layers, 65 x 40 mm, 58 parts, among them J101 USB_B, J102 ISP, J103 IDC, Q101 AO3400A, SW101 BOOT, U101 HPM5301IEG1, U102 USBLC6-2SC6, U103 ISO7741, U104 ISO7741, U105 SN74LVC1G125DBV, U107 RT9193, Y101 24MHz

Commit message: update hardware
Parts:
- removed C127: 0.1uF, Capacitor_SMD:C_0603_1608Metric
- removed H105: MountingHole, myLib:MountingHole_3.2mm_M3
- removed J101: USB_B, myLib:USB_B_Lumberg_2411_02_Horizontal
- removed J102: ISP, Connector_PinHeader_2.54mm:PinHeader_1x04_P2.54mm_Vertical
- removed U103, U104: ISO7741, Package_SO:QSOP-16_3.9x4.9mm_P0.635mm
- removed U105: SN74LVC1G125DBV, Package_TO_SOT_SMD:SOT-23-5
- added F1: 500mA, Fuse:Fuse_0805_2012Metric, F.Cu at (78.2, 130.6)
- added J1: USB_C_Receptacle_USB2.0_16P, akaLinkIso:USB_C_Receptacle_HRO_TYPE-C-31-M-12, F.Cu at (71.5, 129.1)
- added J2: ISP, Connector_PinHeader_2.54mm:PinHeader_1x05_P2.54mm_Vertical, F.Cu at (51.2, 134.9)
- added J3: Conn_JTAG_10, Connector_PinHeader_1.27mm:PinHeader_2x05_P1.27mm_Vertical, F.Cu at (58.0, 135.7)
- added R1: 5.1K, Resistor_SMD:R_0603_1608Metric, F.Cu at (74.0, 135.8)
- added R2: 5.1K, Resistor_SMD:R_0603_1608Metric, F.Cu at (69.0, 135.8)
- added U1: 74LVC1G126, Package_TO_SOT_SMD:SOT-23-5, F.Cu at (74.2, 156.1)
- added U2: ISO6741, Package_SO:SOIC-16W_7.5x10.3mm_P1.27mm, F.Cu at (81.7, 150.4)
- added U3: ISO6741, Package_SO:SOIC-16W_7.5x10.3mm_P1.27mm, F.Cu at (61.3, 150.4)
- H101, H102, H103, H104: footprint myLib:MountingHole_2.2mm_M2 -> akaLinkIso:MountingHole_2.5mm
- J103: footprint Connector_IDC:IDC-Header_2x10_P2.54mm_Horizontal -> akaLinkIso:IDC-Header_2x10_P2.54mm_Horizontal
- L101: footprint Inductor_SMD:L_Sunlord_SWPA4020S -> Inductor_SMD:L_Sunlord_SWPA252012S
- moved H103 171.6 mm to (53.5, 157.0)
- moved C128 161.7 mm to (65.1, 157.6), turned to 180 degrees
- moved J103 156.6 mm to (82.9, 160.6), turned to -90 degrees
- moved R102 156.5 mm to (67.5, 156.1)
- moved Q101 156.5 mm to (70.2, 156.1)
- moved C125 154.0 mm to (71.5, 158.6), turned to 180 degrees
- moved R105 149.9 mm to (80.8, 157.6)
- moved C126 146.8 mm to (85.6, 157.6), turned to 180 degrees
- moved H102 144.4 mm to (83.0, 130.0)
- moved C103 141.2 mm to (65.8, 142.2)
- moved C104 139.6 mm to (68.5, 147.0), turned to 180 degrees
- moved C110 139.1 mm to (62.5, 97.1), turned to 0 degrees
- moved C108 137.4 mm to (62.5, 94.6), turned to 0 degrees
- moved L101 136.2 mm to (71.5, 148.2)
- moved C107 135.9 mm to (62.5, 92.1), turned to 0 degrees
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Connections:
- net /HOSCI renamed /OSCI
- net /HOSCO renamed /OSCO
- D101 pad 1: GND1 -> GND
- R107 pad 1: VCC -> /LED2
- R109 pad 1: +3V3 -> /LED1
- SW101 pad 1: /BOOT1 -> /BL_KEY
- U101 pad 1: unconnected-(U101B-PA04-Pad1) -> /DBG_JTDO
- U101 pad 2: /UART_TXD -> /JTDI_TXD
- U101 pad 20: /nRESET -> /AUX_TXD
- U101 pad 21: /JTRST -> /AUX_RXD
- U101 pad 22: /JTDI -> /LED2
- U101 pad 23: /JTDO -> /LED1
- U101 pad 24: unconnected-(U101B-PB11-Pad24) -> /ADC_VREF
- U101 pad 25: unconnected-(U101B-PB10-Pad25) -> GND
- U101 pad 26: unconnected-(U101B-PB09-Pad26) -> GND
- U101 pad 27: unconnected-(U101B-PB08-Pad27) -> GND
- U101 pad 3: /UART_RXD -> /JTDO_RXD
- U101 pad 37: unconnected-(U101B-PA31-Pad37) -> /JTRST
- U101 pad 4: unconnected-(U101B-PA10-Pad4) -> /BL_KEY
- U101 pad 42: unconnected-(U101B-PA26-Pad42) -> /nRESET
- U101 pad 46: unconnected-(U101B-PA07-Pad46) -> /DBG_JTMS
- U101 pad 47: unconnected-(U101B-PA06-Pad47) -> /DBG_JTCK
- U101 pad 48: unconnected-(U101B-PA05-Pad48) -> /DBG_JTDI
- U102 pad 1: Net-(J101-D-) -> /USB-
- U102 pad 3: Net-(J101-D+) -> /USB+
- U102 pad 5: +5V -> Net-(U102-VBUS)
Routing:
- net +3V3: track 157.7 -> 0.00 mm, vias 12 -> 0
- net VDD_SOC: track 87.6 -> 0.00 mm, vias 5 -> 0
- net VCC: track 59.4 -> 0.00 mm, vias 6 -> 0
- net unconnected-(U101B-PA07-Pad46): track 48.4 -> 0.00 mm, vias 2 -> 0
- net /JTCK: track 42.3 -> 0.00 mm, vias 3 -> 0
- net /ISP_RX: track 37.2 -> 0.00 mm, vias 2 -> 0
- net +5V: track 36.8 -> 0.00 mm, vias 2 -> 0
- net /ISP_TX: track 35.1 -> 0.00 mm, vias 2 -> 0
- net GND: track 34.9 -> 0.00 mm, vias 59 -> 0
- net GND1: track 31.3 -> 0.00 mm, vias 16 -> 0
- net /JTMS_IN: track 30.1 -> 0.00 mm, vias 2 -> 0
- net /JTMS_OUT: track 29.8 -> 0.00 mm, vias 2 -> 0
- net /nRESET: track 28.4 -> 0.00 mm, vias 2 -> 0
- net /JTMS_DIR: track 28.3 -> 0.00 mm, vias 2 -> 0
- net /JTDO: track 22.6 -> 0.00 mm, vias 2 -> 0
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- removed copper zone on F.Cu, net /SW
- removed copper zone on B.Cu, net GND
- removed copper zone on F.Cu, net GND
- removed copper zone on B.Cu, net GND1
- removed copper zone on F.Cu, net GND1
- removed copper zone on F.Cu, net VDD_SOC
Other:
- board size 65 x 40 mm -> 45 x 45 mm
- board text added: "JTAG"
- board text added: "SWD+VCOM"
- board text added: "VREF NC NC GND TXD GND DIO GND CLK GND NC GND RXD NC SRST NC NC NC NC NC"
- board text added: "VREF NC TRST GND TDI GND TMS GND TCK GND NC GND TDO NC SRST NC NC NC NC NC"
- board text added: "akaLink-Iso Rev A.0 @2026/08/17"
- board text removed: "BOOT"
- board text removed: "DuckWang@25/11/09"
- board text removed: "G"
- board text removed: "HSLink-ISO"
- board text removed: "ISO PWR"
- board text removed: "ISP"
- board text removed: "MCU PWR"
- board text removed: "R"
- board text removed: "RUN CON"
- board text removed: "Rev1.0"
- board text removed: "T"
- board text removed: "V"
- board text removed: "VREF NC TRST GND JTDI GND JTMS GND JTCK GND NC GND JTDO DTR SRST RTS NC TXD NC RXD"
