File: hardware/akaLinkPro.kicad_pcb (KiCad board)
At the start: 2 copper layers, 45 x 45 mm, 60 parts, among them J1 USB_C_Receptacle_USB2.0_16P, J103 IDC, J2 ISP, J3 Conn_JTAG_10, Q101 AO3400A, SW101 BOOT, U1 74LVC1G126, U101 HPM5301IEG1, U102 USBLC6-2SC6, U107 RT9193, U2 ISO6741, U3 ISO6741, Y101 24MHz

Commit message: update pcb name
Parts:
- H101, H102, H103, H104: footprint akaLinkIso:MountingHole_2.5mm -> akaLink:MountingHole_2.5mm
- J1: footprint akaLinkIso:USB_C_Receptacle_HRO_TYPE-C-31-M-12 -> akaLink:USB_C_Receptacle_HRO_TYPE-C-31-M-12
- J103: footprint akaLinkIso:IDC-Header_2x10_P2.54mm_Horizontal -> akaLink:IDC-Header_2x10_P2.54mm_Horizontal
