File: hardware_pro/HSLinkIsolate.kicad_pcb (KiCad board)
At the start: 2 copper layers, 45 x 45 mm, 86 parts, among them J1 USB_C_Receptacle_USB2.0_16P, J103 IDC, J2 ISP, J3 TC2050, Q1 SI2305, Q104 AO3400A, Q2 AO3400A, SW101 BL, U1 XC6206P332MR, U101 HPM5301IEG1, U102 USBLC6-2SC6, U105 TPS22918DBV, U110 SN74LVC1T45DBV, U111 SN74LVC1T45DBV, U112 SN74LVC1T45DBV, U113 SN74LVC1T45DBV, U2 LMV321, Y101 24MHz

Commit message: update hardware
Parts:
- C103: footprint Capacitor_SMD:C_0805_2012Metric -> Capacitor_SMD:C_0603_1608Metric
- moved C103 12.4 mm to (71.8, 148.6), turned to -90 degrees
- moved C119 8.01 mm to (79.5, 133.3), turned to 180 degrees
- moved F1 7.90 mm to (85.3, 134.1), turned to 180 degrees
- moved J2 7.40 mm to (50.8, 142.3)
- moved C122 6.39 mm to (85.3, 141.3), turned to 180 degrees
- moved C123 5.18 mm to (85.3, 135.6), turned to 180 degrees
- moved Y101 5.01 mm to (79.5, 135.8), turned to 0 degrees
- moved C115 4.60 mm to (79.5, 142.1)
- moved U1 4.19 mm to (85.3, 138.4), turned to 90 degrees
- moved C120 3.83 mm to (76.6, 135.8), turned to 90 degrees
- moved C116 3.10 mm to (79.5, 145.1)
- moved C130 3.10 mm to (79.5, 140.6)
- moved C118 2.05 mm to (63.4, 140.6)
- moved C101 1.80 mm to (75.0, 148.8)
- moved C102 1.80 mm to (77.0, 148.8)
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
Commit message: update pcb
Parts:
- added C11: 0.1uF, akaLinkIso:C_0603_1608Metric, F.Cu at (63.0, 152.0)
- added C15: 0.1uF, akaLinkIso:C_0603_1608Metric, F.Cu at (63.0, 157.4)
- added R12: 22R, akaLinkIso:R_0603_1608Metric, F.Cu at (63.0, 158.7)
- added R13: 4.7K, akaLinkIso:R_0603_1608Metric, F.Cu at (55.2, 148.3)
- added R14: 4.7K, akaLinkIso:R_0603_1608Metric, F.Cu at (80.0, 152.0)
- added U3: SN74LVC1T45DBV, Package_TO_SOT_SMD:SOT-23-6, F.Cu at (63.0, 154.7)
- C1, C10, C106, C108, C110, C114, C115, C116, C117, C118, C119, C12, C120, C121, C122, C123, C125, C129, C13, C130, C131, C139, C14, C144, C2, C3, C4, C5, C6, C7, C8, C9: footprint Capacitor_SMD:C_0603_1608Metric -> akaLinkIso:C_0603_1608Metric
- C103: footprint Capacitor_SMD:C_0603_1608Metric -> Capacitor_SMD:C_0805_2012Metric
- R1, R10, R101, R103, R104, R107, R109, R11, R110, R113, R117, R125, R127, R128, R129, R130, R133, R2, R3, R4, R5, R6, R7, R8, R9: footprint Resistor_SMD:R_0603_1608Metric -> akaLinkIso:R_0603_1608Metric
- moved R103 13.3 mm to (66.0, 135.8), turned to 90 degrees
- moved C1 11.8 mm to (76.6, 150.7), turned to 180 degrees
- moved C101 10.3 mm to (64.7, 149.7)
- moved C102 10.3 mm to (66.7, 149.7)
- moved R104 9.51 mm to (63.4, 139.1), turned to 180 degrees
- moved R133 8.31 mm to (79.3, 150.1), turned to -90 degrees
- moved C121 6.90 mm to (60.8, 145.1), turned to 180 degrees
- moved R125 5.81 mm to (56.0, 152.8)
- moved R101 4.96 mm to (60.8, 146.4), turned to 180 degrees
- moved R117 4.31 mm to (80.0, 148.1), turned to 180 degrees
- moved C108 3.44 mm to (76.6, 149.4), turned to 0 degrees
- moved C4 3.44 mm to (59.6, 152.0)
- moved U105 3.42 mm to (59.6, 154.7)
- moved R110 3.42 mm to (57.2, 152.8)
- moved R113 3.41 mm to (59.6, 157.4)
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Connections:
- J103 pad 17: unconnected-(J103-Pin_17-Pad17) -> /O_COMRX
Routing:
- net +3V3: track 0.00 -> 27.4 mm, vias 0 -> 1
- net VDD_SOC: track 0.00 -> 24.2 mm
- net /OSCI: track 0.00 -> 9.32 mm
- net /DBG_JTMS: track 0.00 -> 6.73 mm
- net /DBG_JTCK: track 0.00 -> 6.42 mm
- net /OSCO: track 0.00 -> 5.81 mm
- net /DBG_JTDI: track 0.00 -> 5.23 mm
- net /OTPCAP: track 0.00 -> 4.79 mm
- net /DBG_JTDO: track 0.00 -> 4.09 mm
- net /BOOT0: track 0.00 -> 3.25 mm, vias 0 -> 1
- net /JTDI_TXD: track 0.00 -> 3.19 mm, vias 0 -> 1
- net /SW: track 0.00 -> 3.14 mm
- net /USB_D-: track 0.00 -> 3.13 mm
- net /JTDO_RXD: track 0.00 -> 3.05 mm, vias 0 -> 1
- net /BOOT1: track 0.00 -> 3.03 mm, vias 0 -> 1
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Other:
- board text added: "VREF NC NC GND TXD GND DIO GND CLK GND NC GND RXD NC SRST NC VRX NC 5V0 NC"
- board text added: "VREF NC TRST GND TDI GND TMS GND TCK GND NC GND TDO NC SRST NC VRX NC 5V0 NC"
- board text removed: "VREF NC NC GND TXD GND DIO GND CLK GND NC GND RXD NC SRST NC NC NC NC NC"
- board text removed: "VREF NC TRST GND TDI GND TMS GND TCK GND NC GND TDO NC SRST NC NC NC NC NC"
