File: hardware_pro/HSLinkIsolate.kicad_sch (KiCad schematic)
At the start: 86 parts, among them J1 USB_C_Receptacle_USB2.0_16P, J103 IDC, J2 ISP, J3 TC2050, Q1 SI2305, Q104 AO3400A, Q2 AO3400A, SW101 BL, U1 XC6206P332MR, U101 HPM5301IEG1, U102 USBLC6-2SC6, U105 TPS22918DBV, U110 SN74LVC1T45DBV, U111 SN74LVC1T45DBV, U112 SN74LVC1T45DBV, U113 SN74LVC1T45DBV, U2 LMV321, Y101 24MHz

Commit message: update hardware
Parts:
- C103: footprint Capacitor_SMD:C_0805_2012Metric -> Capacitor_SMD:C_0603_1608Metric
Changed lines of the file:
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@@
 			)
 		)
-		(property "Footprint" "Capacitor_SMD:C_0805_2012Metric"
+		(property "Footprint" "Capacitor_SMD:C_0603_1608Metric"
 			(at 63.1952 57.15 0)
 			(effects

Commit message: update pcb
Parts:
- added C11: 0.1uF, akaLinkIso:C_0603_1608Metric, symbol Device:C
- added C15: 0.1uF, akaLinkIso:C_0603_1608Metric, symbol akaLinkCompact:C
- added R12: 22R, akaLinkIso:R_0603_1608Metric, symbol akaLinkCompact:R
- added R13, R14: 4.7K, akaLinkIso:R_0603_1608Metric, symbol akaLinkCompact:R
- added U3: SN74LVC1T45DBV, Package_TO_SOT_SMD:SOT-23-6, symbol akaLinkCompact:SN74LVC1T45DBV
- C1, C10, C106, C108, C110, C114, C115, C116, C117, C118, C119, C12, C120, C121, C122, C123, C125, C129, C13, C130, C131, C139, C14, C144, C2, C3, C4, C5, C6, C7, C8, C9: footprint Capacitor_SMD:C_0603_1608Metric -> akaLinkIso:C_0603_1608Metric
- C103: footprint Capacitor_SMD:C_0603_1608Metric -> Capacitor_SMD:C_0805_2012Metric
- R1, R10, R101, R103, R104, R107, R109, R11, R110, R113, R117, R125, R127, R128, R129, R130, R133, R2, R3, R4, R5, R6, R7, R8, R9: footprint Resistor_SMD:R_0603_1608Metric -> akaLinkIso:R_0603_1608Metric
Connections:
- net +3V3: now also C11.1, U3.1 (VCCA)
- net AUX_RXD: now also U3.3 (A)
- net GND: now also C11.2, C15.2, R13.1, R14.1, U3.2 (GND), U3.5 (DIR)
- net JTRST: now also R14.2
- net VEE: now also C15.1, U3.6 (VCCB)
- net nRESET: now also R13.2
- net O_COMRX: now reaches J103.17 (Pin_17)
- net O_COMRX: now also R12.2
- new net: R12.1, U3.4 (B)
- no-connect marks 15 -> 13
Other:
- moved on the sheet: C4, Q104, Q2, R10, R11, R125, R3, R9
