File: hardware_pro/akaLinkPro.kicad_pcb (KiCad board)
At the start: 2 copper layers, 45 x 45 mm, 92 parts, among them J1 USB_C_Receptacle_USB2.0_16P, J103 IDC, J2 ISP, J3 TC2050, Q1 SI2305, Q104 AO3400A, Q2 AO3400A, SW101 BL, U1 XC6206P332MR, U101 HPM5301IEG1, U102 USBLC6-2SC6, U105 TPS22918DBV, U110 SN74LVC1T45DBV, U111 SN74LVC1T45DBV, U112 SN74LVC1T45DBV, U113 SN74LVC1T45DBV, U2 LMV321, U3 SN74LVC1T45DBV, Y101 24MHz

Commit message: update pcb name
Parts:
- C1, C10, C106, C108, C11, C110, C114, C115, C116, C117, C118, C119, C12, C120, C121, C122, C123, C125, C129, C13, C130, C131, C139, C14, C144, C15, C2, C3, C4, C5, C6, C7, C8, C9: footprint akaLinkIso:C_0603_1608Metric -> akaLink:C_0603_1608Metric
- H101, H102, H103, H104: footprint akaLinkIso:MountingHole_2.5mm -> akaLink:MountingHole_2.5mm
- J1: footprint akaLinkIso:USB_C_Receptacle_HRO_TYPE-C-31-M-12 -> akaLink:USB_C_Receptacle_HRO_TYPE-C-31-M-12
- J103: footprint akaLinkIso:IDC-Header_2x10_P2.54mm_Horizontal -> akaLink:IDC-Header_2x10_P2.54mm_Horizontal
- R1, R10, R101, R103, R104, R107, R109, R11, R110, R113, R117, R12, R125, R127, R128, R129, R13, R130, R133, R14, R2, R3, R4, R5, R6, R7, R8, R9: footprint akaLinkIso:R_0603_1608Metric -> akaLink:R_0603_1608Metric

Commit message: update pcb
Parts:
- removed J3: TC2050, Connector:Tag-Connect_TC2050-IDC-NL_2x05_P1.27mm_Vertical
- removed Q2: AO3400A, Package_TO_SOT_SMD:SOT-23-3
- removed R14, R9: 4.7K, akaLink:R_0603_1608Metric
- added C104: 0.1uF, akaLink:C_0603_1608Metric, F.Cu at (75.5, 150.1)
- added C105: 0.1uF, akaLink:C_0603_1608Metric, F.Cu at (64.0, 145.6)
- added C107: 0.1uF, akaLink:C_0603_1608Metric, F.Cu at (72.2, 149.3)
- added C109: 0.1uF, akaLink:C_0603_1608Metric, F.Cu at (78.9, 143.0)
- added C111: 0.1uF, akaLink:C_0603_1608Metric, F.Cu at (80.0, 152.0)
- added C112: 0.1uF, akaLink:C_0603_1608Metric, F.Cu at (80.0, 157.4)
- added J101: Conn_02x05_Odd_Even, Connector_PinHeader_2.54mm:PinHeader_2x05_P2.54mm_Vertical, F.Cu at (54.9, 134.6)
- added U103: SN74LVC1T45DBV, Package_TO_SOT_SMD:SOT-23-6, F.Cu at (80.0, 154.7)
- moved C121 5.44 mm to (63.4, 149.9), turned to -90 degrees
- moved SW101 5.02 mm to (64.5, 130.5)
- moved R101 3.72 mm to (62.0, 149.9), turned to -90 degrees
- moved R103 2.83 mm to (64.0, 137.8), turned to 180 degrees
- moved R13 1.88 mm to (56.6, 149.6)
- moved Q104 1.77 mm to (59.3, 149.6)
- moved C103 1.60 mm to (73.8, 149.7)
- moved C106 1.00 mm to (64.0, 144.3)
- moved C131 0.94 mm to (78.9, 144.3)
- moved C117 0.85 mm to (64.0, 143.0)
- moved C1 0.80 mm to (77.4, 150.7)
- moved C108 0.80 mm to (77.4, 149.4)
- moved C116 0.80 mm to (78.9, 145.6)
- moved C115 0.74 mm to (78.9, 141.7)
- moved C129 0.72 mm to (64.0, 141.7)
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Connections:
- U110 pad 5: VEE -> +3V3
- U112 pad 5: VEE -> +3V3
Routing:
- net VDD_SOC: track 24.2 -> 0.00 mm
- net +3V3: track 27.4 -> 4.97 mm, vias 1 -> 0
- net /OSCI: track 9.32 -> 0.00 mm
- net /nRST: track 0.64 -> 8.66 mm
- net /DBG_JTMS: track 6.73 -> 0.00 mm
- net /DBG_JTCK: track 6.42 -> 0.00 mm
- net /OSCO: track 5.81 -> 0.00 mm
- net /USB-: track 0.00 -> 5.51 mm
- net /LED1: track 0.00 -> 5.47 mm, vias 0 -> 1
- net /DBG_JTDI: track 5.23 -> 0.00 mm
- net /LED2: track 0.00 -> 5.19 mm, vias 0 -> 1
- net /OTPCAP: track 4.79 -> 0.00 mm
- net /PMCCAP: track 1.92 -> 6.66 mm
- net /AUX_RXD: track 0.00 -> 4.73 mm, vias 0 -> 1
- net /USB+: track 0.00 -> 4.25 mm
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
Commit message: update pcb
Parts:
- removed J101: Conn_02x05_Odd_Even, Connector_PinHeader_2.54mm:PinHeader_2x05_P2.54mm_Vertical
- added J3: TC2050, Connector:Tag-Connect_TC2050-IDC-NL_2x05_P1.27mm_Vertical, F.Cu at (57.5, 139.8)
- moved R104 5.84 mm to (62.8, 144.8), turned to -90 degrees
- moved SW101 5.33 mm to (63.6, 135.8)
- moved R103 4.65 mm to (64.7, 142.4)
- moved C105 1.35 mm to (64.7, 146.8)
- moved C117 1.35 mm to (64.7, 144.2)
- moved C106 1.35 mm to (64.7, 145.4)
- moved C121 1.30 mm to (62.0, 149.9), turned to 90 degrees
- moved R101 1.30 mm to (63.4, 149.9)
- moved C1 1.23 mm to (78.0, 149.7), turned to -90 degrees
- moved J2 1.02 mm to (50.8, 141.2)
- moved C118 0.92 mm to (64.7, 139.8)
- moved C129 0.92 mm to (64.7, 141.1)
- moved C108 0.70 mm to (76.8, 149.7), turned to -90 degrees
- moved C109 0.63 mm to (78.3, 142.8)
- moved C115 0.63 mm to (78.3, 141.4)
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Connections:
- J2 pad 3: /ISP_TX -> /ISP_RX
- J2 pad 4: /ISP_RX -> /ISP_TX
- U101 pad 22: /LED2 -> /5V_EN
- U101 pad 23: /LED1 -> /LED2
- U101 pad 24: /ADC_VREF -> /LED1
- U101 pad 25: /5V_EN -> /ADC_VREF
- U101 pad 47: /DBG_JTCK -> GND
Routing:
- net +3V3: track 4.97 -> 118.8 mm, vias 0 -> 11
- net VDD_SOC: track 0.00 -> 85.2 mm, vias 0 -> 7
- net VEE: track 0.00 -> 56.5 mm, vias 0 -> 8
- net +5V: track 0.00 -> 51.9 mm, vias 0 -> 2
- net /JTRST: track 3.01 -> 47.8 mm, vias 1 -> 2
- net /5V_EN: track 0.00 -> 42.1 mm, vias 0 -> 2
- net /LED2: track 5.19 -> 46.3 mm, vias 1 -> 2
- net /JTMS_DIR: track 3.83 -> 42.0 mm, vias 1 -> 2
- net /JTMS_IN: track 3.92 -> 41.1 mm, vias 1 -> 2
- net /JTCK: track 3.59 -> 37.4 mm, vias 1 -> 2
- net /JTDI_TXD: track 0.00 -> 32.7 mm, vias 0 -> 2
- net /AUX_RXD: track 4.73 -> 35.4 mm, vias 1 -> 2
- net /nRST: track 8.66 -> 36.6 mm, vias 0 -> 2
- net /JTDO_RXD: track 0.00 -> 27.7 mm, vias 0 -> 2
- net /nRESET: track 3.24 -> 28.7 mm, vias 1 -> 2
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- added copper zone on B.Cu, net GND
- added copper zone on F.Cu, net GND

Commit message: update pcb
Parts:
- removed J2: ISP, Connector_PinHeader_2.54mm:PinHeader_1x05_P2.54mm_Vertical
- removed SW101: BL, Button_Switch_SMD:SW_SPST_B3U-1000P
- added J101: ISP, Connector_PinHeader_2.54mm:PinHeader_1x06_P2.54mm_Vertical, F.Cu at (50.8, 138.7)
Connections:
- U101 pad 4: /BL_KEY -> /DFU_PIN
Routing:
- net /DFU_PIN: track 0.00 -> 32.5 mm
- net +3V3: track 118.8 -> 137.0 mm, vias 11 -> 13
- net +5V: track 51.9 -> 67.9 mm
- net Net-(U102-VBUS): track 14.5 -> 27.9 mm
- net /BL_KEY: track 8.72 -> 0.00 mm
- net /nRST: track 36.6 -> 29.0 mm
- net /LED2: track 46.3 -> 49.2 mm
- net VDD_SOC: track 85.2 -> 86.6 mm
- net /DBG_JTMS: track 23.4 -> 24.5 mm
- net /5V_EN: track 42.1 -> 42.9 mm
- net /nRESET: track 28.7 -> 29.3 mm
- net /DBG_JTDI: track 15.0 -> 14.5 mm
- net GND: vias 30 -> 44

Commit message: update hardware
Parts:
- moved C122 1.50 mm to (83.1, 141.6)
- moved U1 1.47 mm to (83.1, 138.9)
- moved C123 1.45 mm to (83.1, 136.2)
- moved F1 1.45 mm to (83.1, 134.8)
Connections:
- J3 pad 4: GND -> /DBG_JTCK
- U101 pad 47: GND -> /DBG_JTCK
Routing:
- net VDD_SOC: track 86.6 -> 60.6 mm, vias 7 -> 9
- net /DBG_JTCK: track 0.00 -> 13.6 mm, vias 0 -> 1
- net GND: track 14.6 -> 7.40 mm
- net +3V3: track 137.0 -> 143.4 mm, vias 13 -> 14
- net /SW: track 2.49 -> 0.10 mm
- net /nRST: track 29.0 -> 27.5 mm
- net +5V: track 67.9 -> 66.8 mm
- net Net-(U102-VBUS): track 27.9 -> 27.3 mm
- added copper zone on F.Cu, net /SW
- added copper zone on F.Cu, net VDD_SOC

Commit message: update pcb
Parts:
- removed J3: TC2050, Connector:Tag-Connect_TC2050-IDC-NL_2x05_P1.27mm_Vertical
- added J102: JTAG, akaLink:PinHeader_2x05_P1.27mm_Vertical, F.Cu at (56.5, 137.4)
- moved R2 4.59 mm to (65.4, 133.0)
- moved C122 1.81 mm to (84.9, 141.8)
- moved C123 1.81 mm to (84.9, 136.4)
- moved F1 1.81 mm to (84.9, 135.0)
- moved U1 1.81 mm to (84.9, 139.1)
- moved C114 1.25 mm to (69.1, 135.7)
- moved C2 0.20 mm to (86.5, 148.2)
Routing:
- net /DBG_JTMS: track 24.5 -> 16.2 mm
- net /CC2: track 2.03 -> 10.1 mm, vias 0 -> 2
- net VDD_SOC: track 60.6 -> 54.1 mm, vias 9 -> 10
- net /nRST: track 27.5 -> 21.9 mm, vias 2 -> 1
- net GND: track 7.40 -> 4.10 mm, vias 44 -> 75
- net /DBG_JTDO: track 16.6 -> 14.7 mm
- net /DBG_JTDI: track 14.5 -> 16.3 mm, vias 0 -> 1
- net /DBG_JTCK: track 13.6 -> 15.2 mm, vias 1 -> 0
- net Net-(U102-VBUS): track 27.3 -> 28.2 mm
- net +3V3: track 143.4 -> 144.2 mm, vias 14 -> 15
- net /ISP_RX: track 19.8 -> 20.4 mm
- added copper zone on B.Cu, net +3V3
- added copper zone on F.Cu, net +3V3
Other:
- board text removed: "akaLink-Pro Rev A.0 @2026/08/18"

Commit message: finish hardware
Routing:
- net +3V3: track 144.2 -> 145.7 mm, vias 15 -> 14
- net VEE: track 56.6 -> 57.5 mm
- net /O_SRST: track 16.6 -> 16.0 mm
- net GND: vias 75 -> 141
Other:
- board text added: "3V3"
- board text added: "BOOT"
- board text added: "DFU"
- board text added: "GND"
- board text added: "RX"
- board text added: "TX"
- board text added: "akaLink Pro Designed by akako Rev A.0@2026/08/30"
