File: hardware_pro/akaLinkPro.kicad_sch (KiCad schematic)
At the start: 92 parts, among them J1 USB_C_Receptacle_USB2.0_16P, J103 IDC, J2 ISP, J3 TC2050, Q1 SI2305, Q104 AO3400A, Q2 AO3400A, SW101 BL, U1 XC6206P332MR, U101 HPM5301IEG1, U102 USBLC6-2SC6, U105 TPS22918DBV, U110 SN74LVC1T45DBV, U111 SN74LVC1T45DBV, U112 SN74LVC1T45DBV, U113 SN74LVC1T45DBV, U2 LMV321, U3 SN74LVC1T45DBV, Y101 24MHz

Commit message: update pcb name
Parts:
- C1, C10, C106, C108, C11, C110, C114, C115, C116, C117, C118, C119, C12, C120, C121, C122, C123, C125, C129, C13, C130, C131, C139, C14, C144, C15, C2, C3, C4, C5, C6, C7, C8, C9: footprint akaLinkIso:C_0603_1608Metric -> akaLink:C_0603_1608Metric
- H101, H102, H103, H104: footprint akaLinkIso:MountingHole_2.5mm -> akaLink:MountingHole_2.5mm
- J1: footprint akaLinkIso:USB_C_Receptacle_HRO_TYPE-C-31-M-12 -> akaLink:USB_C_Receptacle_HRO_TYPE-C-31-M-12
- J103: footprint akaLinkIso:IDC-Header_2x10_P2.54mm_Horizontal -> akaLink:IDC-Header_2x10_P2.54mm_Horizontal
- R1, R10, R101, R103, R104, R107, R109, R11, R110, R113, R117, R12, R125, R127, R128, R129, R13, R130, R133, R14, R2, R3, R4, R5, R6, R7, R8, R9: footprint akaLinkIso:R_0603_1608Metric -> akaLink:R_0603_1608Metric

Commit message: update pcb
Parts:
- removed J3: TC2050, Connector:Tag-Connect_TC2050-IDC-NL_2x05_P1.27mm_Vertical, symbol Connector:TC2050
- removed Q2: AO3400A, Package_TO_SOT_SMD:SOT-23-3, symbol akaLinkCompact:AO3400A
- removed R14, R9: 4.7K, akaLink:R_0603_1608Metric, symbol akaLinkCompact:R
- added C104, C105, C107, C109, C111: 0.1uF, akaLink:C_0603_1608Metric, symbol Device:C
- added C112: 0.1uF, akaLink:C_0603_1608Metric, symbol akaLinkCompact:C
- added J101: Conn_02x05_Odd_Even, Connector_PinHeader_2.54mm:PinHeader_2x05_P2.54mm_Vertical, symbol Connector_Generic:Conn_02x05_Odd_Even
- added U103: SN74LVC1T45DBV, Package_TO_SOT_SMD:SOT-23-6, symbol akaLinkCompact:SN74LVC1T45DBV
Connections:
- net +3V3: now also U110.5 (DIR), U112.5 (DIR), C107.1, C109.1, C111.1, U103.1 (VCCA), U103.5 (DIR)
- net GND: now also C104.2, C105.2, C107.2, C109.2, C111.2, C112.2, U103.2 (GND)
- net JTRST: now also U103.3 (A)
- net OTPCAP: now also C105.1
- net PMCCAP: now also C104.1
- net VEE: now also C112.1, U103.6 (VCCB); no longer U110.5 (DIR), U112.5 (DIR)
- net at R3.1: now also U103.4 (B)
Other:
- moved on the sheet: C10, C103, C11, C110, C114, C115, C116, C117, C118, C125, C129, C130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

Commit message: update pcb
Parts:
- removed J101: Conn_02x05_Odd_Even, Connector_PinHeader_2.54mm:PinHeader_2x05_P2.54mm_Vertical, symbol Connector_Generic:Conn_02x05_Odd_Even
- added J3: TC2050, Connector:Tag-Connect_TC2050-IDC-NL_2x05_P1.27mm_Vertical, symbol Connector:TC2050
Connections:
- net DBG_JTCK is gone; now on net GND: U101.47 (PA06)
- net +3V3: now also J3.1
- net 5V_EN: now also U101.22 (PB13); no longer U101.25 (PB10)
- net ADC_VREF: now also U101.25 (PB10); no longer U101.24 (PB11)
- net DBG_JTDI: now also J3.8
- net DBG_JTDO: now also J3.6
- net DBG_JTMS: now also J3.2
- net GND: now also J3.3, J3.4
- net ISP_RX: now also J2.3 (Pin_3); no longer J2.4 (Pin_4)
- net ISP_TX: now also J2.4 (Pin_4); no longer J2.3 (Pin_3)
- net LED1: now also U101.24 (PB11); no longer U101.23 (PB12)
- net LED2: now also U101.23 (PB12); no longer U101.22 (PB13)
- net nRST: now also J3.10
- no-connect marks 13 -> 16
Other:
- moved on the sheet: C10, C11, C111, C112, C119, C120, C121, C139, C144, C15, C3, C5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

Commit message: update pcb
Parts:
- removed J2: ISP, Connector_PinHeader_2.54mm:PinHeader_1x05_P2.54mm_Vertical, symbol Connector_Generic:Conn_01x05
- removed SW101: BL, Button_Switch_SMD:SW_SPST_B3U-1000P, symbol Switch:SW_Push
- added J101: ISP, Connector_PinHeader_2.54mm:PinHeader_1x06_P2.54mm_Vertical, symbol Connector_Generic:Conn_01x06
Connections:
- net +3V3: now also J101.2 (Pin_2)
- net BOOT1: now also J101.3 (Pin_3)
- net GND: now also J101.6 (Pin_6)
- net ISP_RX: now also J101.4 (Pin_4)
- net ISP_TX: now also J101.5 (Pin_5)
- net BL_KEY renamed DFU_PIN
- net DFU_PIN: now also J101.1 (Pin_1)
Changed lines of the file:
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@@
 	(wire
 		(pts
-			(xy 36.83 234.95) (xy 36.83 237.49)
-		)
-		(stroke
-			(width 0)
-			(type default)
-		)
-	)
-	(wire
-		(pts
 			(xy 130.81 248.92) (xy 130.81 242.57)
 		)
@@
 	(wire
 		(pts
-			(xy 140.97 171.45) (xy 154.94 171.45)
+			(xy 143.51 171.45) (xy 154.94 171.45)
 		)
 		(stroke
@@
 	(wire
 		(pts
-			(xy 36.83 237.49) (xy 34.29 237.49)
+			(xy 43.18 237.49) (xy 34.29 237.49)
 		)
 		(stroke
@@
 	(wire
 		(pts
+			(xy 34.29 234.95) (xy 43.18 234.95)
+		)
+		(stroke
+			(width 0)
+			(type default)
+		)
+	)
+	(wire
+		(pts
 			(xy 212.09 38.1) (xy 212.09 40.64)
 		)
@@
 		)
 	)
-	(label "BL_KEY"
+	(label "DFU_PIN"
 		(at 143.51 171.45 0)
 		(effects
@@
 		)
 	)
+	(label "DFU_PIN"
+		(at 43.18 234.95 180)
+		(effects
+			(font
+				(size 1.27 1.27)
+			)
+			(justify right bottom)
+		)
+	)
 	(label "OTPCAP"
 		(at 125.73 49.53 180)
@@
 	)
 	(symbol
+		(lib_id "Connector_Generic:Conn_01x06")
+		(at 29.21 240.03 0)
+		(mirror y)
+		(unit 1)
+		(exclude_from_sim no)
+		(in_bom no)
+		(on_board yes)
+		(dnp yes)
+		(fields_autoplaced yes)
+		(property "Reference" "J101"
+			(at 29.21 228.6 0)
+			(effects
+				(font
+					(size 1.27 1.27)
+				)
+			)
+		)
+		(property "Value" "ISP"
+			(at 29.21 231.14 0)
+			(effects
+				(font
+					(size 1.27 1.27)
+				)
+			)
+		)
+		(property "Footprint" "Connector_PinHeader_2.54mm:PinHeader_1x06_P2.54mm_Vertical"
+			(at 29.21 240.03 0)
+			(effects
+				(font
+					(size 1.27 1.27)
+				)
+				(hide yes)
+			)
+		)
+		(property "Datasheet" "~"
+			(at 29.21 240.03 0)
+			(effects
+				(font
+					(size 1.27 1.27)
+				)
+				(hide yes)
+			)
+		)
+		(property "Description" "Generic connector, single row, 01x06, script generated (kicad-library-utils/schlib/autogen/connector/)"
+			(at 29.21 240.03 0)
+			(effects
+				(font
+					(size 1.27 1.27)
+				)
+				(hide yes)
+			)
+		)
+		(pin "6"
+		)
+		(pin "4"
+		)
+		(pin "5"
+		)
+		(pin "1"
+		)
+		(pin "2"
+		)
+		(pin "3"
+		)
+		(instances
+			(project "akaLinkPro"
+				(path "/bdacb043-f14a-42d1-8c71-fc9028f33716"
+					(reference "J101")
+					(unit 1)
+				)
+			)
+		)
+	)
+	(symbol
 		(lib_id "power:GND")
 		(at 222.25 48.26 0)
@@
 	)
 	(symbol
-		(lib_id "Switch:SW_Push")
-		(at 135.89 171.45 0)
-		(mirror y)
-		(unit 1)
-		(exclude_from_sim no)
-		(in_bom yes)
-		(on_board yes)
-		(dnp no)
-		(fields_autoplaced yes)
-		(property "Reference" "SW101"
-			(at 135.89 173.99 0)
-			(effects
-				(font
-					(size 1.27 1.27)
-				)
-			)
-		)
-		(property "Value" "BL"
-			(at 135.89 176.53 0)
-			(effects
-				(font
-					(size 1.27 1.27)
-				)
-			)
-		)
-		(property "Footprint" "Button_Switch_SMD:SW_SPST_B3U-1000P"
-			(at 135.89 166.37 0)
-			(effects
-				(font
-					(size 1.27 1.27)
-				)
-				(hide yes)
-			)
-		)
-		(property "Datasheet" "~"
-			(at 135.89 166.37 0)
-			(effects
-				(font
-					(size 1.27 1.27)
-				)
-				(hide yes)
-			)
-		)
-		(property "Description" "Push button switch, generic, two pins"
-			(at 135.89 171.45 0)
-			(effects
-				(font
-					(size 1.27 1.27)
-				)
-				(hide yes)
-			)
-		)
-		(pin "1"
-		)
-		(pin "2"
-		)
-		(instances
-			(project "akaLinkPro"
-				(path "/bdacb043-f14a-42d1-8c71-fc9028f33716"
-					(reference "SW101")
-					(unit 1)
-				)
-			)
-		)
-	)
-	(symbol
 		(lib_id "akaLinkCompact:R")
 		(at 346.71 161.29 90)
@@
 	)
 	(symbol
-		(lib_id "power:+3V3")
-		(at 130.81 171.45 90)
-		(unit 1)
-		(exclude_from_sim no)
-		(in_bom yes)
-		(on_board yes)
-		(dnp no)
-		(fields_autoplaced yes)
-		(property "Reference" "#PWR0138"
-			(at 134.62 171.45 0)
-			(effects
-				(font
-					(size 1.27 1.27)
-				)
-				(hide yes)
-			)
-		)
-		(property "Value" "+3V3"
-			(at 127 171.4499 90)
-			(effects
-				(font
-					(size 1.27 1.27)
-				)
-				(justify left)
-			)
-		)
-		(property "Footprint" ""
-			(at 130.81 171.45 0)
-			(effects
-				(font
-					(size 1.27 1.27)
-				)
-				(hide yes)
-			)
-		)
-		(property "Datasheet" ""
-			(at 130.81 171.45 0)
-			(effects
-				(font
-					(size 1.27 1.27)
-				)
-				(hide yes)
-			)
-		)
-		(property "Description" "Power symbol creates a global label with name \"+3V3\""
-			(at 130.81 171.45 0)
-			(effects
-				(font
-					(size 1.27 1.27)
-				)
-				(hide yes)
-			)
-		)
-		(pin "1"
-		)
-		(instances
-			(project "akaLinkPro"
-				(path "/bdacb043-f14a-42d1-8c71-fc9028f33716"
-					(reference "#PWR0138")
-					(unit 1)
-				)
-			)
-		)
-	)
-	(symbol
 		(lib_id "power:GND")
 		(at 133.35 60.96 90)
@@
 	(symbol
 		(lib_id "power:+3V3")
-		(at 36.83 234.95 0)
+		(at 43.18 237.49 270)
 		(unit 1)
 		(exclude_from_sim no)
@@
 		(fields_autoplaced yes)
 		(property "Reference" "#PWR0134"
-			(at 36.83 238.76 0)
+			(at 39.37 237.49 0)
 			(effects
 				(font
@@
 		)
 		(property "Value" "+3V3"
-			(at 36.83 229.87 0)
+			(at 46.99 237.4899 90)
 			(effects
 				(font
 					(size 1.27 1.27)
 				)
+				(justify left)
 			)
 		)
 		(property "Footprint" ""
-			(at 36.83 234.95 0)
+			(at 43.18 237.49 0)
 			(effects
 				(font
@@
 		)
 		(property "Datasheet" ""
-			(at 36.83 234.95 0)
+			(at 43.18 237.49 0)
 			(effects
 				(font
@@
 		)
 		(property "Description" "Power symbol creates a global label with name \"+3V3\""
-			(at 36.83 234.95 0)
+			(at 43.18 237.49 0)
 			(effects
 				(font
@@
 					(unit 1)
 				)
-			)
-		)
-	)
-	(symbol
-		(lib_id "Connector_Generic:Conn_01x05")
-		(at 29.21 242.57 0)
-		(mirror y)
-		(unit 1)
-		(exclude_from_sim no)
-		(in_bom no)
-		(on_board yes)
-		(dnp yes)
-		(fields_autoplaced yes)
-		(property "Reference" "J2"
-			(at 29.21 231.14 0)
-			(effects
-				(font
-					(size 1.27 1.27)
-				)
-			)
-		)
-		(property "Value" "ISP"
-			(at 29.21 233.68 0)
-			(effects
-				(font
-					(size 1.27 1.27)
-				)
-			)
-		)
-		(property "Footprint" "Connector_PinHeader_2.54mm:PinHeader_1x05_P2.54mm_Vertical"
-			(at 29.21 242.57 0)
-			(effects
-				(font
-					(size 1.27 1.27)
-				)
-				(hide yes)
-			)
-		)
-		(property "Datasheet" "~"
-			(at 29.21 242.57 0)
-			(effects
-				(font
-					(size 1.27 1.27)
-				)
-				(hide yes)
-			)
-		)
-		(property "Description" "Generic connector, single row, 01x05, script generated (kicad-library-utils/schlib/autogen/connector/)"
-			(at 29.21 242.57 0)
-			(effects
-				(font
-					(size 1.27 1.27)
-				)
-				(hide yes)
-			)
-		)
-		(pin "5"
-		)
-		(pin "3"
-		)
-		(pin "2"
-		)
-		(pin "1"
-		)
-		(pin "4"
-		)
-		(instances
-			(project "akaLinkPro"
-				(path "/bdacb043-f14a-42d1-8c71-fc9028f33716"
-					(reference "J2")
-					(unit 1)
-				)

Commit message: update hardware
Connections:
- net GND: no longer J3.4, U101.47 (PA06)
- new net DBG_JTCK: J3.4, U101.47 (PA06)
Other:
- note removed: "JTAG Interface"
- note removed: "LEDs"
- note removed: "MCU IO"
- note removed: "MCU Power"
- note removed: "UART2"
- note removed: "USB Interface"
- moved on the sheet: C1, C10, C101, C102, C103, C104, C105, C106, C107, C108, C109, C11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

Commit message: update pcb
Parts:
- removed J3: TC2050, Connector:Tag-Connect_TC2050-IDC-NL_2x05_P1.27mm_Vertical, symbol Connector:TC2050
- added J102: JTAG, akaLink:PinHeader_2x05_P1.27mm_Vertical, symbol Connector:Conn_ARM_JTAG_SWD_10
Connections:
- net +3V3: now also J102.1 (VTref)
- net DBG_JTCK: now also J102.4 (SWCLK/TCK)
- net DBG_JTDI: now also J102.8 (NC/TDI)
- net DBG_JTDO: now also J102.6 (SWO/TDO)
- net DBG_JTMS: now also J102.2 (SWDIO/TMS)
- net GND: now also J102.3 (GND), J102.5 (GND), J102.9 (GNDDetect)
- net nRST: now also J102.10 (~{RESET})
- no-connect marks 16 -> 13
Other:
- moved on the sheet: D101, D103, J101, R107, R109

Commit message: finish hardware
Other:
- moved on the sheet: C10, C11, C111, C7, C8, C9, F1, J1, J101, J102, R1, R2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
